File: Hardware/SparkFun_Si7021_Breakout.brd (EAGLE design)
At the start: 15.2 x 15.2 mm, 14 parts, among them U1 SI7021

Commit message: Changed version number on BRD and SCH to v10
Other:
- board text added: "v10"
- board text removed: "v01"
Changed lines of the file:
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@@
 <text x="2.667" y="12.065" size="1.016" layer="21" font="vector" ratio="15" rot="R270">-</text>
 <text x="17.78" y="-8.89" size="1.778" layer="51" font="vector">J. Bartlett</text>
-<text x="9.271" y="0.508" size="1.27" layer="16" ratio="20" rot="MR0">v01</text>
+<text x="9.271" y="0.508" size="1.27" layer="16" ratio="20" rot="MR0">v10</text>
 <text x="7.0104" y="6.9596" size="0.8128" layer="21" font="vector" ratio="15" rot="SR90">PU</text>
 <text x="8.4582" y="2.3622" size="0.8128" layer="21" font="vector" ratio="15" rot="R180">Humidity &amp;
