File: Hardware/SparkFun_Si7021_Breakout.sch (EAGLE design)
At the start: 14 parts, among them U1 SI7021

Commit message: Changed version number on BRD and SCH to v10
Other:
- note added: "v10"
- note removed: "v01"
Changed lines of the file:
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@@
 <text x="109.22" y="66.04" size="1.778" layer="97">I2C write is 0x80</text>
 <text x="109.22" y="63.5" size="1.778" layer="97">I2C read is 0x81</text>
-<text x="238.76" y="7.62" size="2.54" layer="94">v01</text>
+<text x="238.76" y="7.62" size="2.54" layer="94">v10</text>
 <text x="43.18" y="119.38" size="1.778" layer="97">Input Voltage Range (VDD): 1.9V to 3.6V</text>
 <text x="50.8" y="116.84" size="1.778" layer="97">I2C Input Voltage Max: VDD</text>
